File: Strobe_main.kicad_pcb (KiCad board)
At the start: 4 copper layers, 100 x 100 mm, 197 parts, among them J1001 Header, J301 10146581-060_M, J302 T44007, J303 T44007, J304 10146581-060_M, J305 T44007, J306 T44007, J501 HX JN1.27-2x5P ZZ H4.9, J502 Header, J701 ZHOURI DC3, J801 Molex 430452427, J901 Header, Q301 MPF3N150, Q302 IXYH55N120, Q303 IXYH55N120, Q304 IXYH55N120, Q305 IXYH55N120, U103 LM217MDT, U104 LM217MDT, U201 AMS1117-3.3, U301 IRS2184, U401 TSV912IDT, U402 TSV912IDT, U403 TSV912IDT, U501 STM32G431K8Tx, U601 ISO1541, U602 ISO6741, Y501 20 MHz

Commit message: Started update of mfg docs
Parts:
- moved C101 135.0 mm to (188.8, 57.2)
- moved C102 135.0 mm to (196.0, 66.5)
- moved C103 135.0 mm to (204.0, 72.5)
- moved C104 135.0 mm to (205.0, 60.0)
- moved C105 135.0 mm to (192.2, 60.0)
- moved C201 135.0 mm to (178.8, 55.8)
- moved C202 135.0 mm to (172.7, 58.8)
- moved C301 135.0 mm to (214.5, 122.6)
- moved C302 135.0 mm to (211.0, 116.5)
- moved C303 135.0 mm to (172.0, 132.5)
- moved C304 135.0 mm to (201.8, 112.2)
- moved C307 135.0 mm to (234.0, 67.2)
- moved C308 135.0 mm to (244.8, 76.0)
- moved C309 135.0 mm to (234.0, 72.5)
- moved C310 135.0 mm to (215.2, 114.5)
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Other:
- board text removed: "30°"

Commit message: Updating mfg docs
Other:
- board text removed: "3× 120°"

Commit message: added 3d model for J501
Other:
- board text removed: "All dimensions are in millimeters unless otherwise specified."
- board text removed: "Impedance Table"
