File: Block Diagram.kicad_sch (KiCad schematic)
At the start: 48 parts, among them J1001 Header, J701 ZHOURI DC3, J801 Molex 430452427, J901 Header

Commit message: Sch update in progress
Parts:
- removed P9: ~, symbol personal:Cosmetic_OUT
Connections:
- net Im_SH1000 renamed Im_S1k
- net SH1000 renamed S1k
- net Um_SH1000: no longer names the net of J801.2 (Pin_2)
- no-connect marks 12 -> 13
Other:
- sheet Lamp driver ports: added LMP_EN, Mon_IL, Mon_LMP, Mon_S1k, S1k; removed Im_Pulse, Lamp_EN, SH1000, Um_Col, Um_Lmp
- sheet MCU ports: added I_S1k, LMP_EN, Mon_IL_prot, Mon_LMP_buf, Mon_S1k_buf, U_S1k_buf; removed I_P_buf, I_SH1000, Lamp_EN, U_C_buf, U_L_buf, U_SH1000_buf
- sheet Signal conditioning ports: added I_S1k, Im_S1k, Mon_IL, Mon_IL_prot, Mon_LMP, Mon_LMP_buf, Mon_S1k, Mon_S1k_buf, U_S1k_buf; removed I_P_buf, I_SH1000, Im_Pulse, Im_SH1000, U_C_buf, U_L_buf, U_SH1000_buf, Um_Col, Um_Lmp, Um_SH1000
Changed lines of the file:
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@@
 	)
 	(junction
-		(at 77.47 165.1)
-		(diameter 0)
-		(color 0 0 0 0)
-	)
-	(junction
 		(at 57.15 199.39)
 		(diameter 0)
@@
 	)
 	(no_connect
+		(at 71.12 179.07)
+	)
+	(no_connect
 		(at 57.15 184.15)
 	)
@@
 	(wire
 		(pts
-			(xy 77.47 165.1) (xy 77.47 179.07)
-		)
-		(stroke
-			(width 0)
-			(type default)
-		)
-	)
-	(wire
-		(pts
 			(xy 99.06 184.15) (xy 99.06 186.69)
 		)
@@
 	(wire
 		(pts
-			(xy 77.47 179.07) (xy 71.12 179.07)
-		)
-		(stroke
-			(width 0)
-			(type default)
-		)
-	)
-	(wire
-		(pts
 			(xy 46.99 191.77) (xy 58.42 191.77)
 		)
@@
 	(wire
 		(pts
-			(xy 77.47 134.62) (xy 121.92 134.62)
-		)
-		(stroke
-			(width 0)
-			(type default)
-		)
-	)
-	(wire
-		(pts
 			(xy 73.66 199.39) (xy 72.39 199.39)
 		)
@@
 	(wire
 		(pts
-			(xy 77.47 134.62) (xy 77.47 165.1)
-		)
-		(stroke
-			(width 0)
-			(type default)
-		)
-	)
-	(wire
-		(pts
 			(xy 71.12 184.15) (xy 85.09 184.15)
 		)
@@
 		)
 	)
-	(label "SH1000"
+	(label "S1k"
 		(at 41.91 184.15 0)
 		(effects
@@
 		)
 	)
-	(label "Um_SH1000"
-		(at 96.52 134.62 0)
-		(effects
-			(font
-				(size 1.27 1.27)
-			)
-			(justify left bottom)
-		)
-	)
 	(label "SL3"
 		(at 289.56 92.71 0)
@@
 		)
 	)
-	(label "SH1000"
+	(label "S1k"
 		(at 55.88 91.44 180)
 		(effects
@@
 		)
 	)
-	(label "Im_SH1000"
+	(label "Im_S1k"
 		(at 96.52 129.54 0)
 		(effects
@@
 	)
 	(symbol
-		(lib_id "personal:Cosmetic_OUT")
-		(at 77.47 165.1 90)
-		(mirror x)
-		(unit 1)
-		(exclude_from_sim no)
-		(in_bom no)
-		(on_board no)
-		(dnp no)
-		(property "Reference" "P9"
-			(at 76.454 165.1 0)
-			(effects
-				(font
-					(size 1.27 1.27)
-				)
-				(hide yes)
-			)
-		)
-		(property "Value" "~"
-			(at 77.47 161.29 0)
-			(effects
-				(font
-					(size 1.27 1.27)
-				)
-				(justify right)
-				(hide yes)
-			)
-		)
-		(property "Footprint" ""
-			(at 77.47 165.1 0)
-			(effects
-				(font
-					(size 1.27 1.27)
-				)
-				(hide yes)
-			)
-		)
-		(property "Datasheet" ""
-			(at 77.47 165.1 0)
-			(effects
-				(font
-					(size 1.27 1.27)
-				)
-				(hide yes)
-			)
-		)
-		(property "Description" ""
-			(at 77.47 165.1 0)
-			(effects
-				(font
-					(size 1.27 1.27)
-				)
-				(hide yes)
-			)
-		)
-		(property "Config" ""
-			(at 77.47 165.1 0)
-			(effects
-				(font
-					(size 1.27 1.27)
-				)
-				(hide yes)
-			)
-		)
-		(property "Manufacturer" ""
-			(at 77.47 165.1 0)
-			(effects
-				(font
-					(size 1.27 1.27)
-				)
-				(hide yes)
-			)
-		)
-		(property "Manufacturer Part Number" ""
-			(at 77.47 165.1 0)
-			(effects
-				(font
-					(size 1.27 1.27)
-				)
-				(hide yes)
-			)
-		)
-		(pin "1"
-		)
-		(instances
-			(project "Strobe_main"
-				(path "/f9e05184-c88b-4a88-ae9c-ab2bdb32be7c/82da9dbf-ba38-4d08-ba35-a220fa2963b1"
-					(reference "P9")
-					(unit 1)
-				)
-			)
-		)
-	)
-	(symbol
 		(lib_id "Connector:Conn_01x03_Pin")
 		(at 347.98 177.8 0)
@@
 			)
 		)
-		(pin "U_L_buf" output
+		(pin "Mon_S1k_buf" output
 			(at 160.02 113.03 0)
 			(effects
@@
 			)
 		)
-		(pin "U_C_buf" output
+		(pin "Mon_LMP_buf" output
 			(at 160.02 115.57 0)
 			(effects
@@
 			)
 		)
-		(pin "I_P_buf" output
+		(pin "Mon_IL_prot" output
 			(at 160.02 118.11 0)
 			(effects
@@
 			)
 		)
-		(pin "Um_Col" input
+		(pin "Mon_LMP" input
 			(at 121.92 115.57 180)
 			(effects
@@
 			)
 		)
-		(pin "Im_Pulse" input
+		(pin "Mon_IL" input
 			(at 121.92 118.11 180)
 			(effects
@@
 			)
 		)
-		(pin "Um_Lmp" input
+		(pin "Mon_S1k" input
 			(at 121.92 113.03 180)
 			(effects
@@
 			)
 		)
-		(pin "I_SH1000" output
+		(pin "I_S1k" output
 			(at 160.02 134.62 0)
 			(effects
@@
 			)
 		)
-		(pin "Um_SH1000" input
-			(at 121.92 134.62 180)
-			(effects
-				(font
-					(size 1.27 1.27)
-				)
-				(justify left)
-			)
-		)
-		(pin "Im_SH1000" input
+		(pin "Im_S1k" input
 			(at 121.92 129.54 180)
 			(effects
@@
 			)
 		)
-		(pin "U_SH1000_buf" output
+		(pin "U_S1k_buf" output
 			(at 160.02 129.54 0)
 			(effects
@@
 			)
 		)
-		(pin "SH1000" input
+		(pin "S1k" input
 			(at 58.42 92.71 180)
 			(effects
@@
 			)
 		)
-		(pin "Lamp_EN" input
+		(pin "LMP_EN" input
 			(at 96.52 97.79 0)
 			(effects
@@
 			)
 		)
-		(pin "Um_Col" output
+		(pin "Mon_LMP" output
 			(at 96.52 115.57 0)
 			(effects
@@
 			)
 		)
-		(pin "Um_Lmp" output
+		(pin "Mon_S1k" output
 			(at 96.52 113.03 0)
 			(effects
@@
 			)
 		)
-		(pin "Im_Pulse" output
+		(pin "Mon_IL" output
 			(at 96.52 118.11 0)
 			(effects
@@
 			)
 		)
-		(pin "Lamp_EN" output
+		(pin "LMP_EN" output
 			(at 185.42 97.79 180)
 			(effects
@@
 			)
 		)
-		(pin "U_L_buf" input
+		(pin "Mon_S1k_buf" input
 			(at 185.42 113.03 180)
 			(effects
@@
 			)
 		)
-		(pin "U_C_buf" input
+		(pin "Mon_LMP_buf" input
 			(at 185.42 115.57 180)
 			(effects
@@
 			)
 		)
-		(pin "I_P_buf" input
+		(pin "Mon_IL_prot" input
 			(at 185.42 118.11 180)
 			(effects
@@
 			)
 		)
-		(pin "I_SH1000" input
+		(pin "I_S1k" input
 			(at 185.42 134.62 180)
 			(effects
@@
 			)
 		)
-		(pin "U_SH1000_buf" input
+		(pin "U_S1k_buf" input
 			(at 185.42 129.54 180)
 			(effects

Commit message: Sch update in progres
Parts:
- removed P10, P12, P13: ~, symbol personal:Cosmetic_OUT
- removed P6: ~, symbol personal:Cosmetic_PWR_SRC
- removed P7, P849, P850, P851: ~, symbol personal:Cosmetic_PWR
Connections:
- net SH0: no longer J801.19 (Pin_19)
- net SH20: no longer J801.4 (Pin_4)
- net Vbus_ctrl: now also J801.6 (Pin_6); no longer J801.3 (Pin_3)
- net MCU/SUP_RX: now reaches J801.18 (Pin_18)
- net SH5: now reaches J801.7 (Pin_7)
- net SH5: now also P5.1, P848.1
- removed net AC_L_P: J801.6 (Pin_6), P848.1
- net AC_N_P: no longer names the net of J801.5 (Pin_5)
- net AC_N_P: no longer P5.1
- net Im_S1k: no longer names the net of J801.13 (Pin_13)
- net Im_SH240: no longer names the net of J801.1 (Pin_1)
- net Um_SH240: no longer names the net of J801.14 (Pin_14)
- new net MCU/SUP_TX: J801.19 (Pin_19)
- no-connect marks 13 -> 5
Other:
- sheet HV side supply renamed Power supply
- removed sheet LV side supply
- sheet MCU ports: added SUP_RX, SUP_TX; removed I_S1k, I_SH240, U_S1k_buf, U_SH240_buf
- sheet Power supply: file HV_side_supply.kicad_sch -> Power_supply.kicad_sch
- sheet Power supply ports: added GND, SH5, SL3; removed AC_L_P, AC_N_P
- sheet Signal conditioning ports: added none; removed I_S1k, I_SH240, Im_S1k, Im_SH240, U_S1k_buf, U_SH240_buf, Um_SH240
- moved on the sheet: J801

Commit message: Sch update complete, ERC OK
Parts:
- removed J801: Molex 430452427, Connector_Molex:Molex_Micro-Fit_3.0_43045-2412_2x12_P3.00mm_Vertical, symbol Connector_Generic:Conn_02x12_Top_Bottom
- added J800: Molex 430451227, Connector_Molex:Molex_Micro-Fit_3.0_43045-1212_2x06_P3.00mm_Vertical, symbol Connector_Generic:Conn_02x06_Top_Bottom
Connections:
- net Earth: now also J800.9 (Pin_9)
- net MCU/SUP_RX: now also J800.1 (Pin_1)
- net MCU/SUP_TX: now also J800.2 (Pin_2)
- net S1k: now also J800.6 (Pin_6)
- net SH0: now also J800.3 (Pin_3)
- net SH5: now also J800.8 (Pin_8)
- net Vbus_ctrl: now also J800.7 (Pin_7)
Other:
- moved on the sheet: H101, H102, H103, H104, J1001, J701, J901, R701, R702
