File: Block Diagram.kicad_sch (KiCad schematic)
At the start: 38 parts, among them J1 Header, J2 ZHOURI DC3, J3 Header, J4 Molex 430451227

Commit message: Changed to checked, updated fab pdf yaml
Parts:
- J1, J3: MAN (none) -> Generic
- J2: MAN (none) -> ZHOURI; MPN (none) -> DC3-2.54-10PAS
- J4: MAN (none) -> Molex; MPN (none) -> 430451227; Manufacturer (none) -> Molex; Manufacturer Part Number (none) -> 430451227
