File: Strobe_main.kicad_sch (KiCad schematic)
At the start: 0 parts

Commit message: Added PCB
Other:
- note removed: "${SHEET_NAME_10}"
- note removed: "${SHEET_NAME_11}"
- note removed: "${SHEET_NAME_12}"
- note removed: "${SHEET_NAME_13}"
- note removed: "${SHEET_NAME_14}"
- note removed: "${SHEET_NAME_15}"
- note removed: "${SHEET_NAME_16}"
- note removed: "10"
- note removed: "11"
- note removed: "12"
- note removed: "13"
- note removed: "14"
- note removed: "15"
- note removed: "16"
Changed lines of the file:
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@@
 	(title_block
 		(title "${SHEETNAME}")
-		(date "2025-01-12")
+		(date "2025-07-04")
 		(rev "${REVISION}")
 		(company "${COMPANY}")
@@
 	(text "Status: ${VARIANT}"
 		(exclude_from_sim no)
-		(at 222.25 222.25 0)
+		(at 220.98 222.25 0)
 		(effects
 			(font
@@
 		)
 	)
-	(text "13"
-		(exclude_from_sim no)
-		(at 31.75 154.94 0)
-		(effects
-			(font
-				(face "Times New Roman")
-				(size 4 4)
-				(color 0 0 0 1)
-			)
-			(justify right bottom)
-			(href "#13")
-		)
-	)
 	(text "7"
 		(exclude_from_sim no)
@@
 		)
 	)
-	(text "11"
-		(exclude_from_sim no)
-		(at 31.75 139.7 0)
-		(effects
-			(font
-				(face "Times New Roman")
-				(size 4 4)
-				(color 0 0 0 1)
-			)
-			(justify right bottom)
-			(href "#11")
-		)
-	)
-	(text "${SHEET_NAME_12}"
-		(exclude_from_sim no)
-		(at 38.1 147.32 0)
-		(effects
-			(font
-				(face "Times New Roman")
-				(size 4 4)
-				(color 0 0 0 1)
-			)
-			(justify left bottom)
-			(href "#12")
-		)
-	)
 	(text "${SHEET_NAME_8}"
 		(exclude_from_sim no)
@@
 		)
 	)
-	(text "10"
-		(exclude_from_sim no)
-		(at 31.75 132.08 0)
-		(effects
-			(font
-				(face "Times New Roman")
-				(size 4 4)
-				(color 0 0 0 1)
-			)
-			(justify right bottom)
-			(href "#10")
-		)
-	)
 	(text "${SHEET_NAME_2}"
 		(exclude_from_sim no)
@@
 			)
 			(justify right bottom)
-		)
-	)
-	(text "14"
-		(exclude_from_sim no)
-		(at 31.75 162.56 0)
-		(effects
-			(font
-				(face "Times New Roman")
-				(size 4 4)
-				(color 0 0 0 1)
-			)
-			(justify right bottom)
-			(href "#14")
 		)
 	)
@@
 		)
 	)
-	(text "${SHEET_NAME_11}"
-		(exclude_from_sim no)
-		(at 38.1 139.7 0)
-		(effects
-			(font
-				(face "Times New Roman")
-				(size 4 4)
-				(color 0 0 0 1)
-			)
-			(justify left bottom)
-			(href "#11")
-		)
-	)
 	(text "${SHEET_NAME_6}"
 		(exclude_from_sim no)
@@
 	(text "Rev ${REVISION}"
 		(exclude_from_sim no)
-		(at 401.32 30.48 0)
+		(at 401.32 33.02 0)
 		(effects
 			(font
@@
 		)
 	)
-	(text "${SHEET_NAME_15}"
-		(exclude_from_sim no)
-		(at 38.1 170.18 0)
-		(effects
-			(font
-				(face "Times New Roman")
-				(size 4 4)
-				(color 0 0 0 1)
-			)
-			(justify left bottom)
-			(href "#15")
-		)
-	)
 	(text "BOTTOM VIEW"
 		(exclude_from_sim no)
@@
 		)
 	)
-	(text "${SHEET_NAME_14}"
-		(exclude_from_sim no)
-		(at 38.1 162.56 0)
-		(effects
-			(font
-				(face "Times New Roman")
-				(size 4 4)
-				(color 0 0 0 1)
-			)
-			(justify left bottom)
-			(href "#14")
-		)
-	)
-	(text "12"
-		(exclude_from_sim no)
-		(at 31.75 147.32 0)
-		(effects
-			(font
-				(face "Times New Roman")
-				(size 4 4)
-				(color 0 0 0 1)
-			)
-			(justify right bottom)
-			(href "#12")
-		)
-	)
 	(text "2"
 		(exclude_from_sim no)
@@
 	(text "${BOARD_NAME}"
 		(exclude_from_sim no)
-		(at 17.78 30.48 0)
+		(at 17.78 33.02 0)
 		(effects
 			(font
@@
 		)
 	)
-	(text "16"
-		(exclude_from_sim no)
-		(at 31.75 177.8 0)
-		(effects
-			(font
-				(face "Times New Roman")
-				(size 4 4)
-				(color 0 0 0 1)
-			)
-			(justify right bottom)
-			(href "#16")
-		)
-	)
-	(text "${SHEET_NAME_16}"
-		(exclude_from_sim no)
-		(at 38.1 177.8 0)
-		(effects
-			(font
-				(face "Times New Roman")
-				(size 4 4)
-				(color 0 0 0 1)
-			)
-			(justify left bottom)
-			(href "#16")
-		)
-	)
 	(text "${SHEET_NAME_3}"
 		(exclude_from_sim no)
@@
 		)
 	)
-	(text "${SHEET_NAME_10}"
-		(exclude_from_sim no)
-		(at 38.1 132.08 0)
-		(effects
-			(font
-				(face "Times New Roman")
-				(size 4 4)
-				(color 0 0 0 1)
-			)
-			(justify left bottom)
-			(href "#10")
-		)
-	)
 	(text "Index"
 		(exclude_from_sim no)
@@
 		)
 	)
-	(text "${SHEET_NAME_13}"
-		(exclude_from_sim no)
-		(at 38.1 154.94 0)
-		(effects
-			(font
-				(face "Times New Roman")
-				(size 4 4)
-				(color 0 0 0 1)
-			)
-			(justify left bottom)
-			(href "#13")
-		)
-	)
 	(text "6"
 		(exclude_from_sim no)
@@
 		)
 	)
-	(text "15"
-		(exclude_from_sim no)
-		(at 31.75 170.18 0)
-		(effects
-			(font
-				(face "Times New Roman")
-				(size 4 4)
-				(color 0 0 0 1)
-			)
-			(justify right bottom)
-			(href "#15")
-		)
-	)

Commit message: Sch update complete, ERC OK
Other:
- note removed: "${SHEET_NAME_4}"
Changed lines of the file:
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@@
-		)
-	)
-	(text "${SHEET_NAME_4}"
-		(exclude_from_sim no)
-		(at 38.1 86.36 0)
-		(effects
-			(font
-				(face "Times New Roman")
-				(size 4 4)
-				(color 0 0 0 1)
-			)
-			(justify left bottom)
-			(href "#4")
 		)
 	)
@@
 			(project "Strobe_main"
 				(path "/f9e05184-c88b-4a88-ae9c-ab2bdb32be7c"
-					(page "9")
+					(page "8")
 				)
 			)
