File: Lamp_driver.kicad_sch (KiCad schematic)
At the start: 121 parts, among them J20 T44007, J21 T44007, J22 T44007, J23 Conn_01x03_Pin, J24 T44007, Q20 MPF3N150, Q21 IXYH55N120, Q22 IXYH55N120, Q23 IXYH55N120, Q24 MDT7N65, U20 IRS2184

Commit message: Changed to checked, updated fab pdf yaml
Parts:
- C20, C21, C22, C23, C27: MAN (none) -> Generic; Manufacturer CCTC -> Generic; Manufacturer Part Number TCC0603X7R104K500CT -> (none)
- C25, C26, C28, R20, R21, R22, R23, R24, R25, R26, R27, R28, R29, R30, R31, R32, R33, R34, R35, R36, R37, R38, R39, R40, R41, R42, R43, R44, R47: MAN (none) -> Generic
- D20, D21: MAN (none) -> DIODES; MPN (none) -> B360A-13-F
- D22, D23, D24: MAN (none) -> DIODES; MPN (none) -> 1N4148W-7-F
- D25, D26, D27, D28, D32: MAN (none) -> HXY MOSFET; MPN (none) -> BZT52C20
- D29: MAN (none) -> LGE; MPN (none) -> S15M
- D30, D31: MAN (none) -> Jingdao Microelectronics; MPN (none) -> 1SMA5953B
- J20, J21, J22, J24: MAN (none) -> XFCN; MPN (none) -> T44007
- J23: value Conn_01x03_Pin -> Header; MAN (none) -> Generic; Manufacturer (none) -> Generic
- PT20: MAN (none) -> Excelitas Technologies; MPN (none) -> ZS1052-S_HT
- Q20: MAN (none) -> Minos; MPN (none) -> MPF3N150; Manufacturer C42401746 -> Minos
- Q21, Q22, Q23: MAN (none) -> IXYS; MPN (none) -> IXYH55N120
- Q24: MAN (none) -> Minos; MPN (none) -> MDT7N65; Manufacturer (none) -> Minos; Manufacturer Part Number (none) -> MDT7N65
- R45, R46: MAN (none) -> Vishay Intertech; MPN (none) -> WSR3R0200FEA
- U20: MAN (none) -> Infineon; MPN (none) -> IRS2184
