File: MCU.kicad_sch (KiCad schematic)
At the start: 86 parts, among them U60 STM32G431K8Tx, Y60 20 MHz

Commit message: Changed to checked, updated fab pdf yaml
Parts:
- C60, C65, C66, D60, D61, R60, R62, R63, R64, R65: MAN (none) -> Generic
- C61, C62, C63, C64: MAN (none) -> Generic; Manufacturer CCTC -> Generic; Manufacturer Part Number TCC0603X7R104K500CT -> (none)
- U60: MAN (none) -> STMicroelectronics; MPN (none) -> STM32G431K8T6
- Y60: MAN (none) -> Generic; Manufacturer huaxindianzi -> Generic; Manufacturer Part Number CF4020M00018001 -> (none)
